File: HDK/Dashboard-Indicators.kicad_pcb (KiCad board)
At the start: 2 copper layers, 95 x 98 mm, 73 parts, among them J101 Conn_02x08_Odd_Even, J102 Conn_02x04_Odd_Even, Q101 AO3401A, Q102 AO3401A, Q103 AO3401A, Q104 AO3400A, Q105 AO3400A, Q106 AO3400A, Q107 AO3400A, Q108 AO3400A, Q109 AO3400A, Q110 AO3400A, Q111 AO3400A, Q112 AO3400A, U1001 74LVC1G57, U104 AMS1117-5.0, U1101 74LVC1G57, U1401 74LVC1G57, U1501 74LVC1G57, U1601 74LVC1G57, U1801 74LVC1G57, U1901 74LVC1G57, U2001 74LVC1G57, U2101 74LVC1G57, U2201 74LVC1G57, U2301 74LVC1G57, U901 74LVC1G57

Commit message: updated rev2 complete
Parts:
- removed C101, C102: 1u, Capacitor_SMD:C_0805_2012Metric
- removed D801, D802: RGB LED, LED_SMD:LED_RGB_1210
- removed the G*** at (75.0, 60.0)
- removed Q101, Q102, Q103: AO3401A, Package_TO_SOT_SMD:SOT-23-3
- removed Q104, Q105, Q106, Q107, Q108, Q109, Q110, Q111, Q112: AO3400A, Package_TO_SOT_SMD:SOT-23-3
- removed REF** (x4): MountingHole_4.3mm_M4_Pad_TopBottom, MountingHole:MountingHole_4.3mm_M4_Pad_TopBottom
- removed REF** (x4): PinHeader_1x10_P2.54mm_Vertical, NVF-Kicad:2.54mm_1x10V-H
- removed RN201, RN202, RN301, RN302, RN401, RN402, RN501, RN502, RN601, RN602, RN701, RN702, RN801, RN802: 47, Resistor_SMD:R_Array_Concave_4x0603
- removed U1001, U1101, U1401, U1501, U1601, U1801, U1901, U2001, U2101, U2201, U2301, U901: 74LVC1G57, Package_TO_SOT_SMD:SOT-363_SC-70-6
- removed U104: AMS1117-5.0, Package_TO_SOT_SMD:SOT-223-3_TabPin2
- removed kibuzzard-65B612BA: G***, kibuzzard-65B612BA
- removed kibuzzard-65B612BF: G***, kibuzzard-65B612BF
- removed kibuzzard-65B612C4: G***, kibuzzard-65B612C4
- removed kibuzzard-65B61402: G***, kibuzzard-65B61402
- removed kibuzzard-65B61406: G***, kibuzzard-65B61406
- removed kibuzzard-65B61451: G***, kibuzzard-65B61451
- removed kibuzzard-65B6145B: G***, kibuzzard-65B6145B
- added C201: 1u, Capacitor_SMD:C_0805_2012Metric, B.Cu at (77.4, 66.1)
- added C202: 220n, Capacitor_SMD:C_0603_1608Metric, B.Cu at (67.9, 65.5)
- added C301: 1u, Capacitor_SMD:C_0805_2012Metric, B.Cu at (77.4, 76.1)
- added C302: 220n, Capacitor_SMD:C_0603_1608Metric, B.Cu at (67.9, 75.5)
- added C401: 1u, Capacitor_SMD:C_0805_2012Metric, B.Cu at (77.4, 86.1)
- added C402: 220n, Capacitor_SMD:C_0603_1608Metric, B.Cu at (67.9, 85.5)
- added C501: 1u, Capacitor_SMD:C_0805_2012Metric, B.Cu at (77.4, 96.1)
- added C502: 220n, Capacitor_SMD:C_0603_1608Metric, B.Cu at (67.9, 95.5)
- added C601: 1u, Capacitor_SMD:C_0805_2012Metric, B.Cu at (77.4, 106.1)
- added C602: 220n, Capacitor_SMD:C_0603_1608Metric, B.Cu at (67.9, 105.5)
- added C701: 1u, Capacitor_SMD:C_0805_2012Metric, B.Cu at (77.4, 116.1)
- added C702: 220n, Capacitor_SMD:C_0603_1608Metric, B.Cu at (67.9, 115.5)
- added D101: SS14, Diode_SMD:D_SMA, B.Cu at (125.0, 82.0)
- added D102: SS14, Diode_SMD:D_SMA, B.Cu at (125.0, 116.4)
- added D203: LED, LED_THT:LED_Rectangular_W5.0mm_H2.0mm, F.Cu at (58.7, 63.7)
- added D204: LED, LED_THT:LED_Rectangular_W5.0mm_H2.0mm, F.Cu at (55.7, 66.3)
- added D303: LED, LED_THT:LED_Rectangular_W5.0mm_H2.0mm, F.Cu at (58.7, 73.7)
- added D304: LED, LED_THT:LED_Rectangular_W5.0mm_H2.0mm, F.Cu at (55.7, 76.3)
- added D403: LED, LED_THT:LED_Rectangular_W5.0mm_H2.0mm, F.Cu at (58.7, 83.7)
- added D404: LED, LED_THT:LED_Rectangular_W5.0mm_H2.0mm, F.Cu at (55.7, 86.3)
- added D503: LED, LED_THT:LED_Rectangular_W5.0mm_H2.0mm, F.Cu at (58.7, 93.7)
- added D504: LED, LED_THT:LED_Rectangular_W5.0mm_H2.0mm, F.Cu at (55.7, 96.3)
- added D603: LED, LED_THT:LED_Rectangular_W5.0mm_H2.0mm, F.Cu at (58.7, 103.7)
- added D604: LED, LED_THT:LED_Rectangular_W5.0mm_H2.0mm, F.Cu at (55.7, 106.3)
- added D703: LED, LED_THT:LED_Rectangular_W5.0mm_H2.0mm, F.Cu at (58.7, 113.7)
- added D704: LED, LED_THT:LED_Rectangular_W5.0mm_H2.0mm, F.Cu at (55.7, 116.3)
- added G***: LOGO, NVF-Kicad:NVF-Logo-30mm, F.Cu at (90.1, 58.5)
- added G***: LOGO, NVF-Kicad:NVF-Logo-30mm, B.Cu at (89.9, 58.5)
- added H101: MountingHole_Pad, MountingHole:MountingHole_4.3mm_M4_DIN965_Pad_TopBottom, F.Cu at (56.0, 56.0)
- added H102: MountingHole_Pad, MountingHole:MountingHole_4.3mm_M4_DIN965_Pad_TopBottom, F.Cu at (124.0, 56.0)
- added H103: MountingHole_Pad, MountingHole:MountingHole_4.3mm_M4_DIN965_Pad_TopBottom, F.Cu at (56.0, 124.0)
- added H104: MountingHole_Pad, MountingHole:MountingHole_4.3mm_M4_DIN965_Pad_TopBottom, F.Cu at (124.0, 124.0)
- added L201: 22uH, Inductor_SMD:L_1008_2520Metric, B.Cu at (74.4, 66.2)
- added L301: 22uH, Inductor_SMD:L_1008_2520Metric, B.Cu at (74.4, 76.2)
- added L401: 22uH, Inductor_SMD:L_1008_2520Metric, B.Cu at (74.4, 86.2)
- added L501: 22uH, Inductor_SMD:L_1008_2520Metric, B.Cu at (74.4, 96.2)
- added L601: 22uH, Inductor_SMD:L_1008_2520Metric, B.Cu at (74.4, 106.2)
- added L701: 22uH, Inductor_SMD:L_1008_2520Metric, B.Cu at (74.4, 116.2)
- added R101: 4k7, Resistor_SMD:R_0603_1608Metric, B.Cu at (119.0, 72.0)
- added R102: 4k7, Resistor_SMD:R_0603_1608Metric, B.Cu at (119.0, 74.0)
- added R103: 4k7, Resistor_SMD:R_0603_1608Metric, B.Cu at (119.0, 76.0)
- added R104: 4k7, Resistor_SMD:R_0603_1608Metric, B.Cu at (118.2, 107.0)
- added R105: 4k7, Resistor_SMD:R_0603_1608Metric, B.Cu at (118.2, 111.0)
- added R106: 4k7, Resistor_SMD:R_0603_1608Metric, B.Cu at (118.2, 109.0)
- added R107: 1k, Resistor_SMD:R_0603_1608Metric, B.Cu at (114.4, 72.0)
- added R108: 1k, Resistor_SMD:R_0603_1608Metric, B.Cu at (114.4, 74.0)
- added R109: 1k, Resistor_SMD:R_0603_1608Metric, B.Cu at (114.4, 76.0)
- added R110: 1k, Resistor_SMD:R_0603_1608Metric, B.Cu at (113.6, 106.8)
- added R111: 1k, Resistor_SMD:R_0603_1608Metric, B.Cu at (113.6, 111.0)
- added R112: 1k, Resistor_SMD:R_0603_1608Metric, B.Cu at (113.6, 108.8)
- added R201: 10, Resistor_SMD:R_0603_1608Metric, B.Cu at (67.9, 68.7)
- added R301: 10, Resistor_SMD:R_0603_1608Metric, B.Cu at (67.9, 78.7)
- added R401: 10, Resistor_SMD:R_0603_1608Metric, B.Cu at (67.9, 88.7)
- added R501: 10, Resistor_SMD:R_0603_1608Metric, B.Cu at (67.9, 98.7)
- added R601: 10, Resistor_SMD:R_0603_1608Metric, B.Cu at (67.9, 108.7)
- added R701: 10, Resistor_SMD:R_0603_1608Metric, B.Cu at (67.9, 118.7)
- added RV101: R_Potentiometer, Potentiometer_THT:Potentiometer_Bourns_3296W_Vertical, B.Cu at (107.0, 124.2)
- added U201: AP3019A, Package_SO:TSOP-6_1.65x3.05mm_P0.95mm, B.Cu at (70.7, 66.3)
- added U301: AP3019A, Package_SO:TSOP-6_1.65x3.05mm_P0.95mm, B.Cu at (70.7, 76.3)
- added U401: AP3019A, Package_SO:TSOP-6_1.65x3.05mm_P0.95mm, B.Cu at (70.7, 86.3)
- added U501: AP3019A, Package_SO:TSOP-6_1.65x3.05mm_P0.95mm, B.Cu at (70.7, 96.3)
- added U601: AP3019A, Package_SO:TSOP-6_1.65x3.05mm_P0.95mm, B.Cu at (70.7, 106.3)
- added U701: AP3019A, Package_SO:TSOP-6_1.65x3.05mm_P0.95mm, B.Cu at (70.7, 116.3)
- added kibuzzard-65BB44D5: G***, kibuzzard-65BB44D5, F.Cu at (94.0, 86.0)
- added kibuzzard-65BB44FC: G***, kibuzzard-65BB44FC, F.Cu at (94.0, 76.0)
- added kibuzzard-65BB4501: G***, kibuzzard-65BB4501, F.Cu at (94.0, 66.0)
- added kibuzzard-65BB4514: G***, kibuzzard-65BB4514, F.Cu at (94.0, 96.0)
- added kibuzzard-65BB451D: G***, kibuzzard-65BB451D, F.Cu at (94.0, 116.0)
- added kibuzzard-65BB5B6A: G***, kibuzzard-65BB5B6A, F.Cu at (94.0, 106.0)
- added kibuzzard-65BBEAC3: G***, kibuzzard-65BBEAC3, B.Cu at (99.0, 87.2)
- added kibuzzard-65BBEACE: G***, kibuzzard-65BBEACE, B.Cu at (103.2, 95.0)
- D201, D202, D301, D302, D401, D402, D501, D502, D601, D602, D701, D702: value RGB LED -> LED; footprint LED_SMD:LED_RGB_1210 -> LED_THT:LED_Rectangular_W5.0mm_H2.0mm
- J101: value Conn_02x08_Odd_Even -> PHD_02x04V-H; footprint Connector_JST:JST_PHD_B16B-PHDSS_2x08_P2.00mm_Vertical -> NVF-Kicad:PHD_02x04V-H
- J102: value Conn_02x04_Odd_Even -> PHD_02x04V-H; footprint Connector_JST:JST_PHD_B8B-PHDSS_2x04_P2.00mm_Vertical -> NVF-Kicad:PHD_02x04V-H
- moved J102 33.2 mm to (125.0, 108.0), turned to 90 degrees
- moved J101 32.7 mm to (125.0, 73.0), turned to 90 degrees
- moved D501 26.6 mm to (64.7, 93.7)
- moved D601 24.7 mm to (64.7, 103.7)
- moved D502 22.3 mm to (61.7, 96.3), turned to 90 degrees
- moved D602 20.3 mm to (61.7, 106.3), turned to 90 degrees
- moved D701 16.3 mm to (64.7, 113.7)
- moved D702 15.8 mm to (61.7, 116.3), turned to 90 degrees
- moved D401 11.8 mm to (64.7, 83.7)
- moved D201 11.8 mm to (64.7, 63.7)
- moved D301 11.7 mm to (64.7, 73.7)
- moved D202 4.53 mm to (61.7, 66.3), turned to 90 degrees
- moved D402 4.53 mm to (61.7, 86.3), turned to 90 degrees
- moved D302 4.51 mm to (61.7, 76.3), turned to 90 degrees
Connections:
- D201 pad 1: Net-(D201-BA) -> Net-(D201-K)
- D201 pad 2: Net-(D201-GA) -> /TS OFF Indicator/V_{OUT}
- D202 pad 2: Net-(D202-GA) -> Net-(D201-K)
- D301 pad 1: Net-(D301-BA) -> Net-(D301-K)
- D301 pad 2: Net-(D301-GA) -> /AMS FAULT Indicator/V_{OUT}
- D302 pad 2: Net-(D302-GA) -> Net-(D301-K)
- D401 pad 1: Net-(D401-BA) -> Net-(D401-K)
- D401 pad 2: Net-(D401-GA) -> /IMD FAULT Indicator/V_{OUT}
- D402 pad 2: Net-(D402-GA) -> Net-(D401-K)
- D501 pad 1: Net-(D501-BA) -> Net-(D501-K)
- D501 pad 2: Net-(D501-GA) -> /Overtemp Indicator/V_{OUT}
- D502 pad 2: Net-(D502-GA) -> Net-(D501-K)
- D601 pad 1: Net-(D601-BA) -> Net-(D601-K)
- D601 pad 2: Net-(D601-GA) -> /R2D ON Indicator/V_{OUT}
- D602 pad 2: Net-(D602-GA) -> Net-(D601-K)
- D701 pad 1: Net-(D701-BA) -> Net-(D701-K)
- D701 pad 2: Net-(D701-GA) -> /R2D RDY Indicator/V_{OUT}
- D702 pad 2: Net-(D702-GA) -> Net-(D701-K)
- J101 pad 1: +5V -> Net-(D101-A)
- J101 pad 2: VCC -> /IMD FAULT Indicator/CTRL
- J101 pad 3: /R2D_ON -> Net-(D101-A)
- J101 pad 4: /PUMP_ON -> /AMS FAULT Indicator/CTRL
- J101 pad 5: /R2D_RDY -> GND
- J101 pad 6: /PUMP_AUTO -> /TS OFF Indicator/CTRL
- J101 pad 7: /R2D_OFF -> GND
- J101 pad 8: /PUMP_ON_SW -> unconnected-(J101-Pin_8-Pad8)
- J102 pad 1: /TS_ON -> Net-(D102-A)
- J102 pad 2: /AMS_FLT -> /R2D RDY Indicator/CTRL
- J102 pad 3: /TS_ON_N -> Net-(D102-A)
- J102 pad 4: /AMS_FLT_N -> /R2D ON Indicator/CTRL
- J102 pad 5: /IMD_FLT -> GND
- J102 pad 6: VCC -> /Overtemp Indicator/CTRL
- J102 pad 7: /IMD_FLT_N -> GND
- J102 pad 8: GND -> unconnected-(J102-Pin_8-Pad8)
Routing:
- net VCC: track 0.00 -> 223.0 mm, vias 0 -> 14
- net /AMS FAULT Indicator/FB: track 0.00 -> 202.5 mm
- net /Overtemp Indicator/CTRL: track 0.00 -> 62.1 mm
- net /TS OFF Indicator/CTRL: track 0.00 -> 60.1 mm
- net /IMD FAULT Indicator/CTRL: track 0.00 -> 59.1 mm
- net /R2D ON Indicator/CTRL: track 0.00 -> 58.8 mm
- net /R2D RDY Indicator/CTRL: track 0.00 -> 57.3 mm
- net /AMS FAULT Indicator/CTRL: track 0.00 -> 56.9 mm
- net /Indicator-AMS/RED: track 36.4 -> 0.00 mm
- net /PUMP_AUTO_LED: track 35.9 -> 0.00 mm
- net GND: track 0.00 -> 34.9 mm, vias 36 -> 30
- net /AMS_FLTLED: track 33.3 -> 0.00 mm
- net /FAULT_LED: track 33.0 -> 0.00 mm
- net /AMS_FLT_LED: track 31.0 -> 0.00 mm
- net /Indicator-PUMP_AUTO/RED: track 30.4 -> 0.00 mm
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- removed copper zone on F.Cu, net +5V
- removed copper zone on F.Cu, net VCC
Other:
- board size 95 x 98 mm -> 80 x 80 mm
- board text added: "0.0000 mm / 0.0000 mm"
- board text added: "0.3000 mm"
- board text added: "1.6000 mm"
- board text added: "2"
- board text added: "80.0000 mm x 80.0000 mm"
- board text added: "BOARD CHARACTERISTICS"
- board text added: "Board Thickness:"
- board text added: "Board overall dimensions:"
- board text added: "Brightness"
- board text added: "Castellated pads:"
- board text added: "Copper Finish:"
- board text added: "Copper Layer Count:"
- board text added: "Dashboard-Indicators Rev2"
- board text added: "Edge card connectors:"
- board text added: "Impedance Control:"
- board text added: "Min hole diameter:"
- board text added: "Min track/spacing:"
- board text added: "No"
- board text added: "None"
- board text added: "Plated Board Edge:"
- board text added: "Scott CJX"

Commit message: wip
Other:
- board text added: "JLCJLCJLCJLC"
Changed lines of the file:
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@@
     (descr "Resistor SMD 0603 (1608 Metric), square (rectangular) end terminal, IPC_7351 nominal, (Body size source: IPC-SM-782 page 72, https://www.pcb-3d.com/wordpress/wp-content/uploads/ipc-sm-782a_amendment_1_and_2.pdf), generated with kicad-footprint-generator")
     (tags "resistor")
-    (property "LCSC" "C17903")
+    (property "LCSC" "C22859")
     (property "Sheetfile" "Indicator.kicad_sch")
     (property "Sheetname" "AMS FAULT Indicator")
@@
     (descr "Resistor SMD 0603 (1608 Metric), square (rectangular) end terminal, IPC_7351 nominal, (Body size source: IPC-SM-782 page 72, https://www.pcb-3d.com/wordpress/wp-content/uploads/ipc-sm-782a_amendment_1_and_2.pdf), generated with kicad-footprint-generator")
     (tags "resistor")
-    (property "LCSC" "C25819")
+    (property "LCSC" "C23162")
     (property "Sheetfile" "Dashboard-Indicators.kicad_sch")
     (property "Sheetname" "")
@@
     (descr "Resistor SMD 0603 (1608 Metric), square (rectangular) end terminal, IPC_7351 nominal, (Body size source: IPC-SM-782 page 72, https://www.pcb-3d.com/wordpress/wp-content/uploads/ipc-sm-782a_amendment_1_and_2.pdf), generated with kicad-footprint-generator")
     (tags "resistor")
-    (property "LCSC" "C17903")
+    (property "LCSC" "C22859")
     (property "Sheetfile" "Indicator.kicad_sch")
     (property "Sheetname" "IMD FAULT Indicator")
@@
     (descr "Resistor SMD 0603 (1608 Metric), square (rectangular) end terminal, IPC_7351 nominal, (Body size source: IPC-SM-782 page 72, https://www.pcb-3d.com/wordpress/wp-content/uploads/ipc-sm-782a_amendment_1_and_2.pdf), generated with kicad-footprint-generator")
     (tags "resistor")
-    (property "LCSC" "C25819")
+    (property "LCSC" "C23162")
     (property "Sheetfile" "Dashboard-Indicators.kicad_sch")
     (property "Sheetname" "")
@@
     (descr "Resistor SMD 0603 (1608 Metric), square (rectangular) end terminal, IPC_7351 nominal, (Body size source: IPC-SM-782 page 72, https://www.pcb-3d.com/wordpress/wp-content/uploads/ipc-sm-782a_amendment_1_and_2.pdf), generated with kicad-footprint-generator")
     (tags "resistor")
-    (property "LCSC" "C17903")
+    (property "LCSC" "C22859")
     (property "Sheetfile" "Indicator.kicad_sch")
     (property "Sheetname" "R2D RDY Indicator")
@@
     (descr "Resistor SMD 0603 (1608 Metric), square (rectangular) end terminal, IPC_7351 nominal, (Body size source: IPC-SM-782 page 72, https://www.pcb-3d.com/wordpress/wp-content/uploads/ipc-sm-782a_amendment_1_and_2.pdf), generated with kicad-footprint-generator")
     (tags "resistor")
-    (property "LCSC" "C17903")
+    (property "LCSC" "C22859")
     (property "Sheetfile" "Indicator.kicad_sch")
     (property "Sheetname" "R2D ON Indicator")
@@
     (descr "Resistor SMD 0603 (1608 Metric), square (rectangular) end terminal, IPC_7351 nominal, (Body size source: IPC-SM-782 page 72, https://www.pcb-3d.com/wordpress/wp-content/uploads/ipc-sm-782a_amendment_1_and_2.pdf), generated with kicad-footprint-generator")
     (tags "resistor")
-    (property "LCSC" "C25819")
+    (property "LCSC" "C23162")
     (property "Sheetfile" "Dashboard-Indicators.kicad_sch")
     (property "Sheetname" "")
@@
     (descr "Resistor SMD 0603 (1608 Metric), square (rectangular) end terminal, IPC_7351 nominal, (Body size source: IPC-SM-782 page 72, https://www.pcb-3d.com/wordpress/wp-content/uploads/ipc-sm-782a_amendment_1_and_2.pdf), generated with kicad-footprint-generator")
     (tags "resistor")
-    (property "LCSC" "C17903")
+    (property "LCSC" "C22859")
     (property "Sheetfile" "Indicator.kicad_sch")
     (property "Sheetname" "Overtemp Indicator")
@@
     (descr "Resistor SMD 0603 (1608 Metric), square (rectangular) end terminal, IPC_7351 nominal, (Body size source: IPC-SM-782 page 72, https://www.pcb-3d.com/wordpress/wp-content/uploads/ipc-sm-782a_amendment_1_and_2.pdf), generated with kicad-footprint-generator")
     (tags "resistor")
-    (property "LCSC" "C25819")
+    (property "LCSC" "C23162")
     (property "Sheetfile" "Dashboard-Indicators.kicad_sch")
     (property "Sheetname" "")
@@
     (descr "Resistor SMD 0603 (1608 Metric), square (rectangular) end terminal, IPC_7351 nominal, (Body size source: IPC-SM-782 page 72, https://www.pcb-3d.com/wordpress/wp-content/uploads/ipc-sm-782a_amendment_1_and_2.pdf), generated with kicad-footprint-generator")
     (tags "resistor")
-    (property "LCSC" "C25819")
+    (property "LCSC" "C23162")
     (property "Sheetfile" "Dashboard-Indicators.kicad_sch")
     (property "Sheetname" "")
@@
     (descr "Resistor SMD 0603 (1608 Metric), square (rectangular) end terminal, IPC_7351 nominal, (Body size source: IPC-SM-782 page 72, https://www.pcb-3d.com/wordpress/wp-content/uploads/ipc-sm-782a_amendment_1_and_2.pdf), generated with kicad-footprint-generator")
     (tags "resistor")
-    (property "LCSC" "C17903")
+    (property "LCSC" "C22859")
     (property "Sheetfile" "Indicator.kicad_sch")
     (property "Sheetname" "TS OFF Indicator")
@@
     (descr "Resistor SMD 0603 (1608 Metric), square (rectangular) end terminal, IPC_7351 nominal, (Body size source: IPC-SM-782 page 72, https://www.pcb-3d.com/wordpress/wp-content/uploads/ipc-sm-782a_amendment_1_and_2.pdf), generated with kicad-footprint-generator")
     (tags "resistor")
-    (property "LCSC" "C25819")
+    (property "LCSC" "C23162")
     (property "Sheetfile" "Dashboard-Indicators.kicad_sch")
     (property "Sheetname" "")
@@
     )
     (stroke (width 0.15) (type solid)) (fill none) (layer "Edge.Cuts"))
+  (gr_text "JLCJLCJLCJLC" (at 60.2 70.4) (layer "B.SilkS")
+    (effects (font (size 1 1) (thickness 0.15)) (justify mirror))
+  )
   (gr_text "Scott CJX" (at 110 81.6) (layer "B.SilkS")
     (effects (font (size 1.5 1.5) (thickness 0.3) bold) (justify mirror))
