File: HDK/Dashboard-Indicators.kicad_pcb (KiCad board)
At the start: 2 copper layers, 80 x 80 mm, 85 parts, among them J101 PHD_02x04V-H, J102 PHD_02x04V-H, U201 AP3019A, U301 AP3019A, U401 AP3019A, U501 AP3019A, U601 AP3019A, U701 AP3019A

Commit message: final-archive
Parts:
- removed C201, C301, C401, C501, C601, C701: 1u, Capacitor_SMD:C_0805_2012Metric
- removed C202, C302, C402, C502, C602, C702: 220n, Capacitor_SMD:C_0603_1608Metric
- removed D101, D102: SS14, Diode_SMD:D_SMA
- removed D201, D202, D203, D204, D301, D302, D303, D304, D401, D402, D403, D404, D501, D502, D503, D504, D601, D602, D603, D604, D701, D702, D703, D704: LED, LED_THT:LED_Rectangular_W5.0mm_H2.0mm
- removed the G*** at (90.1, 58.5)
- removed the G*** at (89.9, 58.5)
- removed H101, H102, H103, H104: MountingHole_Pad, MountingHole:MountingHole_4.3mm_M4_DIN965_Pad_TopBottom
- removed J101, J102: PHD_02x04V-H, NVF-Kicad:PHD_02x04V-H
- removed L201, L301, L401, L501, L601, L701: 22uH, Inductor_SMD:L_1008_2520Metric
- removed R101, R102, R103, R104, R105, R106: 4k7, Resistor_SMD:R_0603_1608Metric
- removed R107, R108, R109, R110, R111, R112: 1k, Resistor_SMD:R_0603_1608Metric
- removed R201, R301, R401, R501, R601, R701: 10, Resistor_SMD:R_0603_1608Metric
- removed RV101: R_Potentiometer, Potentiometer_THT:Potentiometer_Bourns_3296W_Vertical
- removed U201, U301, U401, U501, U601, U701: AP3019A, Package_SO:TSOP-6_1.65x3.05mm_P0.95mm
- removed kibuzzard-65BB44D5: G***, kibuzzard-65BB44D5
- removed kibuzzard-65BB44FC: G***, kibuzzard-65BB44FC
- removed kibuzzard-65BB4501: G***, kibuzzard-65BB4501
- removed kibuzzard-65BB4514: G***, kibuzzard-65BB4514
- removed kibuzzard-65BB451D: G***, kibuzzard-65BB451D
- removed kibuzzard-65BB5B6A: G***, kibuzzard-65BB5B6A
- removed kibuzzard-65BBEAC3: G***, kibuzzard-65BBEAC3
- removed kibuzzard-65BBEACE: G***, kibuzzard-65BBEACE
- added G***: LOGO, NVF-Kicad:NVF-Logo-30mm, F.Cu at (142.0, 122.5)
- added REF**: LED_D5.0mm, NVF-Kicad:LED_D5.0mm, F.Cu at (132.8, 110.2)
- added REF**: D_SMA, Diode_SMD:D_SMA, B.Cu at (159.0, 110.8)
- added REF**: FUSE-MCCQ-122, NVF-Kicad:FUSE-MCCQ-122, B.Cu at (157.0, 98.2)
- added REF**: R_0603_1608Metric, Resistor_SMD:R_0603_1608Metric, B.Cu at (146.2, 93.3)
- added REF**: R_1206_3216Metric, Resistor_SMD:R_1206_3216Metric, B.Cu at (138.0, 93.5)
- added REF**: LED_D5.0mm, NVF-Kicad:LED_D5.0mm, F.Cu at (132.8, 102.2)
- added REF**: LED_D5.0mm, NVF-Kicad:LED_D5.0mm, F.Cu at (132.8, 94.2)
- added REF**: MountingHole_4.3mm_M4_DIN965_Pad_TopBottom, MountingHole:MountingHole_4.3mm_M4_DIN965_Pad_TopBottom, F.Cu at (159.5, 121.5)
- added REF**: MountingHole_4.3mm_M4_DIN965_Pad_TopBottom, MountingHole:MountingHole_4.3mm_M4_DIN965_Pad_TopBottom, F.Cu at (133.5, 75.0)
- added REF**: LED_D5.0mm, NVF-Kicad:LED_D5.0mm, F.Cu at (132.8, 86.2)
- added REF**: SOT-23, Package_TO_SOT_SMD:SOT-23, B.Cu at (142.5, 93.3)
- added REF**: JST_PH_B8B-PH-SM4-TB_1x08-1MP_P2.00mm_Vertical, Connector_JST:JST_PH_B8B-PH-SM4-TB_1x08-1MP_P2.00mm_Vertical, B.Cu at (140.0, 121.5)
- added REF**: D_SMA, Diode_SMD:D_SMA, B.Cu at (155.0, 110.8)
- added kibuzzard-65CCFF11: G***, kibuzzard-65CCFF11, F.Cu at (144.5, 86.2)
- added kibuzzard-65CCFF21: G***, kibuzzard-65CCFF21, F.Cu at (144.5, 94.2)
- added kibuzzard-65CCFF2A: G***, kibuzzard-65CCFF2A, F.Cu at (144.5, 102.2)
- added kibuzzard-65CD056D: G***, kibuzzard-65CD056D, F.Cu at (150.4, 110.2)
Routing:
- net VCC: track 223.0 -> 0.00 mm, vias 14 -> 0
- net /AMS FAULT Indicator/FB: track 202.5 -> 0.00 mm
- net (no net): track 0.00 -> 96.9 mm, vias 0 -> 2
- net /Overtemp Indicator/CTRL: track 62.1 -> 0.00 mm
- net /TS OFF Indicator/CTRL: track 60.1 -> 0.00 mm
- net /IMD FAULT Indicator/CTRL: track 59.1 -> 0.00 mm
- net /R2D ON Indicator/CTRL: track 58.8 -> 0.00 mm
- net /R2D RDY Indicator/CTRL: track 57.3 -> 0.00 mm
- net /AMS FAULT Indicator/CTRL: track 56.9 -> 0.00 mm
- net GND: track 34.9 -> 0.00 mm, vias 30 -> 0
- net Net-(D101-A): track 8.41 -> 0.00 mm
- net Net-(D102-A): track 7.81 -> 0.00 mm
- net /TS OFF Indicator/V_{OUT}: track 7.02 -> 0.00 mm
- net /R2D RDY Indicator/V_{OUT}: track 6.86 -> 0.00 mm
- net /R2D ON Indicator/V_{OUT}: track 6.86 -> 0.00 mm
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- removed copper zone on B.Cu, net GND
- removed copper zone on F.Cu, net GND
Other:
- board size 80 x 80 mm -> 38.3 x 58.5 mm
- board text removed: "0.0000 mm / 0.0000 mm"
- board text removed: "0.3000 mm"
- board text removed: "1.6000 mm"
- board text removed: "2"
- board text removed: "80.0000 mm x 80.0000 mm"
- board text removed: "BOARD CHARACTERISTICS"
- board text removed: "Board Thickness:"
- board text removed: "Board overall dimensions:"
- board text removed: "Brightness"
- board text removed: "Castellated pads:"
- board text removed: "Copper Finish:"
- board text removed: "Copper Layer Count:"
- board text removed: "Dashboard-Indicators Rev2"
- board text removed: "Edge card connectors:"
- board text removed: "Impedance Control:"
- board text removed: "Min hole diameter:"
- board text removed: "Min track/spacing:"
- board text removed: "No"
- board text removed: "None"
- board text removed: "Plated Board Edge:"
- board text removed: "Scott CJX"
