File: HDK/Dashboard-Indicators.kicad_sch (KiCad schematic)
At the start: 21 parts, among them J101 PHD_02x04V-H, J102 PHD_02x04V-H

Commit message: wip
Parts:
- R101, R102, R103, R104, R105, R106: LCSC C25819 -> C23162
Changed lines of the file:
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@@
       (effects (font (size 1.27 1.27)) hide)
     )
-    (property "LCSC" "C25819" (at 170.18 62.23 0)
+    (property "LCSC" "C23162" (at 170.18 62.23 0)
       (effects (font (size 1.27 1.27)) hide)
     )
@@
       (effects (font (size 1.27 1.27)) hide)
     )
-    (property "LCSC" "C25819" (at 161.29 62.23 0)
+    (property "LCSC" "C23162" (at 161.29 62.23 0)
       (effects (font (size 1.27 1.27)) hide)
     )
@@
       (effects (font (size 1.27 1.27)) hide)
     )
-    (property "LCSC" "C25819" (at 196.85 62.23 0)
+    (property "LCSC" "C23162" (at 196.85 62.23 0)
       (effects (font (size 1.27 1.27)) hide)
     )
@@
       (effects (font (size 1.27 1.27)) hide)
     )
-    (property "LCSC" "C25819" (at 179.07 62.23 0)
+    (property "LCSC" "C23162" (at 179.07 62.23 0)
       (effects (font (size 1.27 1.27)) hide)
     )
@@
       (effects (font (size 1.27 1.27)) hide)
     )
-    (property "LCSC" "C25819" (at 152.4 62.23 0)
+    (property "LCSC" "C23162" (at 152.4 62.23 0)
       (effects (font (size 1.27 1.27)) hide)
     )
@@
       (effects (font (size 1.27 1.27)) hide)
     )
-    (property "LCSC" "C25819" (at 187.96 62.23 0)
-      (effects (font (size 1.27 1.27)) hide)
-    )
+    (property "LCSC" "C23162" (at 187.96 62.23 0)
+      (effects (font (size 1.27 1.27)) hide)
+    )
