File: HDK/Dashboard-Indicators.kicad_sch (KiCad schematic)
At the start: 17 parts, among them J101 Conn_02x08_Odd_Even, J102 Conn_02x04_Odd_Even, Q101 AO3401A, Q102 AO3401A, Q103 AO3401A, Q104 AO3400A, Q105 AO3400A, Q106 AO3400A, Q107 AO3400A, Q108 AO3400A, Q109 AO3400A, Q110 AO3400A, Q111 AO3400A, Q112 AO3400A, U104 AMS1117-5.0

Commit message: updated rev2 complete
Parts:
- removed C101, C102: 1u, Capacitor_SMD:C_0805_2012Metric, symbol Device:C
- removed J101: Conn_02x08_Odd_Even, Connector_JST:JST_PHD_B16B-PHDSS_2x08_P2.00mm_Vertical, symbol Connector_Generic:Conn_02x08_Odd_Even
- removed Q101, Q102, Q103: AO3401A, Package_TO_SOT_SMD:SOT-23-3, symbol Simulation_SPICE:PMOS
- removed Q104, Q105, Q106, Q107, Q108, Q109, Q110, Q111, Q112: AO3400A, Package_TO_SOT_SMD:SOT-23-3, symbol Simulation_SPICE:NMOS
- removed U104: AMS1117-5.0, Package_TO_SOT_SMD:SOT-223-3_TabPin2, symbol Regulator_Linear:AMS1117-5.0
- added D101, D102: SS14, Diode_SMD:D_SMA, symbol Device:D_Schottky
- added H101, H102, H103, H104: MountingHole_Pad, MountingHole:MountingHole_4.3mm_M4_DIN965_Pad_TopBottom, symbol Mechanical:MountingHole_Pad
- added J101: PHD_02x04V-H, NVF-Kicad:PHD_02x04V-H, symbol Connector_Generic:Conn_02x04_Odd_Even
- added R101, R102, R103, R104, R105, R106: 4k7, Resistor_SMD:R_0603_1608Metric, symbol Device:R
- added R107, R108, R109, R110, R111, R112: 1k, Resistor_SMD:R_0603_1608Metric, symbol Device:R
- added RV101: R_Potentiometer, Potentiometer_THT:Potentiometer_Bourns_3296W_Vertical, symbol Device:R_Potentiometer
- J102: value Conn_02x04_Odd_Even -> PHD_02x04V-H; footprint Connector_JST:JST_PHD_B8B-PHDSS_2x04_P2.00mm_Vertical -> NVF-Kicad:PHD_02x04V-H; LCSC (none) -> -
Connections:
- net IMD_FLT is gone; now on net GND: J102.5 (Pin_5)
- net IMD_FLT_N is gone; now on net GND: J102.7 (Pin_7)
- net TS_ON_N is gone; now on an unnamed net: J102.3 (Pin_3)
- net GND: now also H101.1, H102.1, H103.1, H104.1, J101.5 (Pin_5), J101.7 (Pin_7), R107.1, R108.1, R109.1, R110.1, R111.1, R112.1, RV101.3; no longer J102.8 (Pin_8)
- net VCC: now also D101.1 (K), D102.1 (K), R101.2, R102.2, R103.2, R104.2, R105.2, R106.2, RV101.1; no longer J102.6 (Pin_6)
- net AMS_FLT renamed ~{R2D_ON}
- net ~{R2D_ON}: now also R105.1, R111.2
- net AMS_FLT_N renamed ~{R2D_RDY}
- net ~{R2D_RDY}: now also R106.1, R112.2
- net TS_ON: no longer names the net of J102.1 (Pin_1)
- net TS_ON: now also D102.2 (A)
- new net: D101.2 (A), J101.1 (Pin_1), J101.3 (Pin_3)
- new net V_{Brightness}: RV101.2
- new net ~{AMS_FAULT}: J101.4 (Pin_4), R102.1, R108.2
- new net ~{IMD_FAULT}: J101.2 (Pin_2), R103.1, R109.2
- new net ~{TEMP_WARN}: J102.6 (Pin_6), R104.1, R110.2
- new net ~{TS_OFF}: J101.6 (Pin_6), R101.1, R107.2
- no-connect marks 7 -> 2
Other:
- removed sheet AND1
- removed sheet AND2
- removed sheet AND3
- removed sheet Indicator-AMS
- removed sheet Indicator-IMD
- removed sheet Indicator-PUMP_AUTO
- removed sheet Indicator-PUMP_ON
- removed sheet Indicator-R2D_OFF
- removed sheet Indicator-R2D_ON
- removed sheet Indicator-TSAC
- removed sheet SCS_CHK
- removed sheet SCS_CHK1
- removed sheet SCS_CHK2
- added sheet AMS FAULT Indicator (Indicator.kicad_sch)
- added sheet IMD FAULT Indicator (Indicator.kicad_sch)
- added sheet Overtemp Indicator (Indicator.kicad_sch)
- added sheet R2D ON Indicator (Indicator.kicad_sch)
- added sheet R2D RDY Indicator (Indicator.kicad_sch)
- added sheet TS OFF Indicator (Indicator.kicad_sch)
- note added: "Aux Indicators + Handling"
- note added: "SCS Signal Indicators + Handling"
- note added: "SCS Signals are Pulled-Up: Display "Fault" by default"
- note added: "note: ~{TS_OFF} should be ON by default"
- note removed: "AMS Indicators"
- note removed: "Control Connects"
- note removed: "IMD Indicators"
- note removed: "Power + Brightness Control"
- note removed: "Pump Indicators"
- note removed: "R2D Dashboard Controller + Driving of Indicators"
- note removed: "R2D Indicators"
- note removed: "SCS Signal Check + Driving of Indicators"
- note removed: "TSAC Indicators"
- company: (none) -> Scott CJX

Commit message: final-archive
Parts:
- removed D101, D102: SS14, Diode_SMD:D_SMA, symbol Device:D_Schottky
- removed H101, H102, H103, H104: MountingHole_Pad, MountingHole:MountingHole_4.3mm_M4_DIN965_Pad_TopBottom, symbol Mechanical:MountingHole_Pad
- removed J101, J102: PHD_02x04V-H, NVF-Kicad:PHD_02x04V-H, symbol Connector_Generic:Conn_02x04_Odd_Even
- removed R104, R105, R106: 4k7, Resistor_SMD:R_0603_1608Metric, symbol Device:R
- removed R107, R108, R109, R110, R111, R112: 1k, Resistor_SMD:R_0603_1608Metric, symbol Device:R
- removed RV101: R_Potentiometer, Potentiometer_THT:Potentiometer_Bourns_3296W_Vertical, symbol Device:R_Potentiometer
- added D101: LED, symbol Device:LED
- added Q101: Q_NMOS_GSD, symbol Device:Q_NMOS_GSD
- R101: value 4k7 -> 120; footprint Resistor_SMD:R_0603_1608Metric -> (none); LCSC C25819 -> (none)
- R102: value 4k7 -> 10k; footprint Resistor_SMD:R_0603_1608Metric -> (none); LCSC C25819 -> (none)
- R103: value 4k7 -> 1k; footprint Resistor_SMD:R_0603_1608Metric -> (none); LCSC C25819 -> (none)
Connections:
- net ~{AMS_FAULT} is gone; now on net VCC: R102.1
- net GND: now also R103.2, D101.1 (K)
- net VCC: now also Q101.3 (D); no longer R101.2, R102.2, R103.2
- net ~{IMD_FAULT} renamed SIG
- net SIG: now also R102.2, Q101.1 (G)
- net ~{TS_OFF}: no longer names the net of R101.1
- net ~{TS_OFF}: now also Q101.2 (S)
- new net: D101.2 (A), R101.2
- no-connect marks 2 -> 0
Other:
- removed sheet AMS FAULT Indicator
- removed sheet IMD FAULT Indicator
- removed sheet Overtemp Indicator
- removed sheet R2D ON Indicator
- removed sheet R2D RDY Indicator
- removed sheet TS OFF Indicator
- note removed: "Aux Indicators + Handling"
- note removed: "SCS Signal Indicators + Handling"
- note removed: "SCS Signals are Pulled-Up: Display "Fault" by default"
- note removed: "note: ~{TS_OFF} should be ON by default"
