File: HDK/Indicator.kicad_sch (KiCad schematic)
At the start: 17 parts, among them J101 Conn_02x08_Odd_Even, J102 Conn_02x04_Odd_Even, Q101 AO3401A, Q102 AO3401A, Q103 AO3401A, Q104 AO3400A, Q105 AO3400A, Q106 AO3400A, Q107 AO3400A, Q108 AO3400A, Q109 AO3400A, Q110 AO3400A, Q111 AO3400A, Q112 AO3400A, U104 AMS1117-5.0

Commit message: added rev1-cancelled
Parts:
- removed C101, C102: 1u, Capacitor_SMD:C_0805_2012Metric, symbol Device:C
- removed J101: Conn_02x08_Odd_Even, Connector_JST:JST_PHD_B16B-PHDSS_2x08_P2.00mm_Vertical, symbol Connector_Generic:Conn_02x08_Odd_Even
- removed J102: Conn_02x04_Odd_Even, Connector_JST:JST_PHD_B8B-PHDSS_2x04_P2.00mm_Vertical, symbol Connector_Generic:Conn_02x04_Odd_Even
- removed Q101, Q102, Q103: AO3401A, Package_TO_SOT_SMD:SOT-23-3, symbol Simulation_SPICE:PMOS
- removed Q104, Q105, Q106, Q107, Q108, Q109, Q110, Q111, Q112: AO3400A, Package_TO_SOT_SMD:SOT-23-3, symbol Simulation_SPICE:NMOS
- removed U104: AMS1117-5.0, Package_TO_SOT_SMD:SOT-223-3_TabPin2, symbol Regulator_Linear:AMS1117-5.0
- added D? (x2): RGB LED, LED_SMD:LED_RGB_1210, symbol Device:LED_BGKR
- added RN201, RN202: 47, Resistor_SMD:R_Array_Concave_4x0603, symbol NVF-Kicad:R_Network04_Split
Connections:
- net GND: now also D?.3 (K), D?.3 (K)
- new net: D?.1 (BA), RN201.8 (R1.2)
- new net: D?.2 (GA), RN201.7 (R2.2)
- new net: D?.4 (RA), RN201.6 (R3.2)
- new net: D?.4 (RA), RN202.6 (R3.2)
- new net: D?.1 (BA), RN202.8 (R1.2)
- new net: D?.2 (GA), RN202.7 (R2.2)
- new net BLUE: RN201.1 (R1.2), RN202.1 (R1.2)
- new net GREEN: RN201.2 (R1), RN202.2 (R1)
- new net RED: RN201.3 (R3.2), RN202.3 (R3.2)
- no-connect marks 7 -> 0
Other:
- removed sheet AND1
- removed sheet AND2
- removed sheet AND3
- removed sheet Indicator-AMS
- removed sheet Indicator-IMD
- removed sheet Indicator-PUMP_AUTO
- removed sheet Indicator-PUMP_ON
- removed sheet Indicator-R2D_OFF
- removed sheet Indicator-R2D_ON
- removed sheet Indicator-TSAC
- removed sheet SCS_CHK
- removed sheet SCS_CHK1
- removed sheet SCS_CHK2
- note removed: "AMS Indicators"
- note removed: "Control Connects"
- note removed: "IMD Indicators"
- note removed: "Power + Brightness Control"
- note removed: "Pump Indicators"
- note removed: "R2D Dashboard Controller + Driving of Indicators"
- note removed: "R2D Indicators"
- note removed: "SCS Signal Check + Driving of Indicators"
- note removed: "TSAC Indicators"

Commit message: updated rev2 complete
Parts:
- removed D? (x2): RGB LED, LED_SMD:LED_RGB_1210, symbol Device:LED_BGKR
- removed RN201, RN202: 47, Resistor_SMD:R_Array_Concave_4x0603, symbol NVF-Kicad:R_Network04_Split
- added C101: 1u, Capacitor_SMD:C_0805_2012Metric, symbol Device:C
- added C102: 220n, Capacitor_SMD:C_0603_1608Metric, symbol Device:C
- added D101, D102, D103, D104: LED, LED_THT:LED_Rectangular_W5.0mm_H2.0mm, symbol Device:LED
- added L101: 22uH, Inductor_SMD:L_1008_2520Metric, symbol Device:L
- added R108: 10, Resistor_SMD:R_0603_1608Metric, symbol Device:R
- added U101: AP3019A, Package_SO:TSOP-6_1.65x3.05mm_P0.95mm, symbol NVF-Kicad:AP3019A
Connections:
- net GND: now also C101.2, C102.2, R108.2, U101.2 (GND)
- new net: D102.1 (K), D103.2 (A)
- new net: D101.1 (K), D102.2 (A)
- new net: L101.2, U101.1 (SW)
- new net: D103.1 (K), D104.2 (A)
- new net CTRL: U101.4 (CTRL)
- new net VCC: C101.1, L101.1, U101.6 (V_{IN})
- new net V_{Brightness}: D104.1 (K), R108.1, U101.3 (FB)
- new net V_{OUT}: C102.1, D101.2 (A), U101.5 (V_{OUT})
Other:
- company: (none) -> Scott CJX

Commit message: wip
Parts:
- R108: LCSC C17903 -> C22859
Changed lines of the file:
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@@
       (effects (font (size 1.27 1.27)) hide)
     )
-    (property "LCSC" "C17903" (at 67.31 36.83 0)
+    (property "LCSC" "C22859" (at 67.31 36.83 0)
       (effects (font (size 1.27 1.27)) hide)
     )
